File: xmas tree/tree_pcb.brd (EAGLE design)
At the start: 84 x 96 mm, 16 parts

Commit message: back up
Parts:
- added J1: FEMALE_HEADER_8X1, xmas_tree:8X1_HEADER_THT
- moved D1 86.0 mm to (76.0, 8.00), flipped to the top, turned to 0 degrees
- moved D3 50.6 mm to (70.0, 28.0), flipped to the top, turned to 0 degrees
- moved D16 44.8 mm to (43.0, 56.0), flipped to the top
- moved D8 38.6 mm to (50.0, 83.0), flipped to the top
- moved D7 31.4 mm to (48.0, 70.0), flipped to the top
- moved D2 30.6 mm to (67.0, 15.0), flipped to the top, turned to 0 degrees
- moved D14 23.3 mm to (56.0, 25.0), flipped to the top
- moved D4 22.8 mm to (62.0, 36.0), flipped to the top, turned to 0 degrees
- moved D10 19.8 mm to (40.0, 28.0), flipped to the top
- moved D12 19.1 mm to (25.0, 8.00), flipped to the top
- moved D15 18.8 mm to (50.0, 39.0), flipped to the top
- moved D11 18.6 mm to (31.0, 18.0), flipped to the top
- moved D9 13.0 mm to (38.0, 43.0), flipped to the top
- moved D6 11.7 mm to (55.0, 60.0), flipped to the top
- moved D13 11.3 mm to (48.0, 14.0), flipped to the top, turned to 0 degrees
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Connections:
- removed net GND: D1.1
- removed net VCC: D1.2
- new net 1: D1.1, D13.1, D5.1, D9.1, J1.5
- new net 2: D10.1, D14.1, D2.1, D6.1, J1.6
- new net 3: D11.1, D15.1, D3.1, D7.1, J1.7
- new net 4: D12.1, D16.1, D4.1, D8.1, J1.8
- new net A: D1.2, D2.2, D3.2, D4.2, J1.1
- new net B: D5.2, D6.2, D7.2, D8.2, J1.2
- new net C: D10.2, D11.2, D12.2, D9.2, J1.3
- new net D: D13.2, D14.2, D15.2, D16.2, J1.4
Routing:
- net 4: track 0.00 -> 150.5 mm, vias 0 -> 1
- net 2: track 0.00 -> 127.2 mm, vias 0 -> 5
- net 3: track 0.00 -> 119.0 mm, vias 0 -> 4
- net B: track 0.00 -> 116.3 mm
- net 1: track 0.00 -> 96.2 mm, vias 0 -> 3
- net C: track 0.00 -> 75.0 mm
- net A: track 0.00 -> 65.1 mm
- net D: track 0.00 -> 59.4 mm
