File: xmas tree/tree_pcb.brd (EAGLE design)
At the start: 84 x 96 mm, 17 parts, among them J1 FEMALE_HEADER_8X1

Commit message: basic course done
Parts:
- removed D1: red, xmas_tree:SIDE_MOUNT
- removed D10, D11, D12, D13, D14, D15, D16, D2, D3, D4, D5, D6, D7, D8, D9: (no value), xmas_tree:SIDE_MOUNT
- removed J1: FEMALE_HEADER_8X1, xmas_tree:8X1_HEADER_THT
Connections:
- removed net NET_1: D1.1, D13.1, D5.1, D9.1, J1.5
- removed net NET_2: D10.1, D14.1, D2.1, D6.1, J1.6
- removed net NET_3: D11.1, D15.1, D3.1, D7.1, J1.7
- removed net NET_4: D12.1, D16.1, D4.1, D8.1, J1.8
- removed net NET_A: D1.2, D2.2, D3.2, D4.2, J1.1
- removed net NET_B: D5.2, D6.2, D7.2, D8.2, J1.2
- removed net NET_C: D10.2, D11.2, D12.2, D9.2, J1.3
- removed net NET_D: D13.2, D14.2, D15.2, D16.2, J1.4
Routing:
- net NET_4: track 150.5 -> 0.00 mm, vias 1 -> 0
- net NET_2: track 127.2 -> 0.00 mm, vias 5 -> 0
- net NET_3: track 119.0 -> 0.00 mm, vias 4 -> 0
- net NET_B: track 116.3 -> 0.00 mm
- net NET_1: track 96.2 -> 0.00 mm, vias 3 -> 0
- net NET_C: track 75.0 -> 0.00 mm
- net NET_A: track 65.1 -> 0.00 mm
- net NET_D: track 59.4 -> 0.00 mm
