File: xmas tree/tree_pcb.sch (EAGLE design)
At the start: 17 parts, among them J1 FEMALE_HEADER_8X1

Commit message: back up
Parts:
- D1: value (none) -> red
Connections:
- net 1 renamed NET_1
- net 2 renamed NET_2
- net 3 renamed NET_3
- net 4 renamed NET_4
- net A renamed NET_A
- net B renamed NET_B
- net C renamed NET_C
- net D renamed NET_D
Other:
- note added: "Schematic Phase: 1. Add LEDs and Header 2. Set the value of LEDs 3. Connect components 4. Set the name of Nest 5. ERC Check"
- moved on the sheet: D1, D10, D11, D12, D13, D14, D15, D16, D2, D3, D4, D5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

Commit message: basic course done
Parts:
- removed D1: red, xmas_tree:LEDSIDE_MOUNT
- removed D10, D11, D12, D13, D14, D15, D16, D2, D3, D4, D5, D6, D7, D8, D9: (no value), xmas_tree:LEDSIDE_MOUNT
- removed J1: FEMALE_HEADER_8X1, xmas_tree:FEMALE_HEADER_8X1
Connections:
- removed net NET_1: D1.2, D13.2, D5.2, D9.2, J1.5
- removed net NET_2: D10.2, D14.2, D2.2, D6.2, J1.6
- removed net NET_3: D11.2, D15.2, D3.2, D7.2, J1.7
- removed net NET_4: D12.2, D16.2, D4.2, D8.2, J1.8
- removed net NET_A: D1.1, D2.1, D3.1, D4.1, J1.1
- removed net NET_B: D5.1, D6.1, D7.1, D8.1, J1.2
- removed net NET_C: D10.1, D11.1, D12.1, D9.1, J1.3
- removed net NET_D: D13.1, D14.1, D15.1, D16.1, J1.4
